File: MainBoard/MainBoard.kicad_sch (KiCad schematic)
At the start: 43 parts, among them J1 1761681-3, Q1 BC557, U1 LM393, U2 TL074

Commit message: testing
Parts:
- added Q2: BC547, Package_TO_SOT_THT:TO-92_Inline, symbol Transistor_BJT:BC547
- added R14: 10k, symbol Device:R
Connections:
- net Comparator: now also R14.2
- net GND: now also Q2.3 (E)
- net at R7.2, R8.1, R9.1: now also Q2.1 (C); no longer U1.7
- new net: Q2.2 (B), R14.1, U1.7
Other:
- moved on the sheet: C7, D5, D6, D9, Q1, R10, R8, R9, RV1, RV2, RV3, RV4

Commit message: testing
Parts:
- added R16: 10k, symbol Device:R
Connections:
- net +v: now also R16.2
- net at Q2.1 (C), R7.2, R8.1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: now also R16.1
Other:
- note added: ".options method=gear .options gmin=1e-9 cshunt=1e-12 .options reltol=1e-2 abstol=1e-9 vntol=1e-6 .options itl1=300 itl4=300 .options maxstep=100p .options temp=60 .tran 100u 1000ms .control run plot v(Gate) v(Net-_D3-A_) + 0.25 v(Net-_U1A--_) v(Net-_U1A--_, Net-_D3-A_) v(Comparator) plot v(Net-_D9-K_) v(Net-_Q2-B_) + 0.25 v(Envelope) v(Output) plot v(Envelope) v(Net-_U2C--_) + 0.25 v(Feedback) + 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"
- note removed: ".options method=gear .options gmin=1e-9 cshunt=1e-12 .options reltol=1e-2 abstol=1e-9 vntol=1e-6 .options itl1=300 itl4=300 .options maxstep=100p .options temp=60 .tran 100u 1000ms .control run plot v(Gate) v(Net-_D3-A_) + 0.25 v(Net-_U1A--_) v(Net-_U1A--_, Net-_D3-A_) v(Comparator) plot v(Net-_D9-K_) v(Net-_R7-Pad2_) + 0.25 v(Envelope) v(Output) plot v(Envelope) v(Net-_U2C--_) + 0.25 v(Feedback)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"
Changed lines of the file:
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@@
 		)
 	)
-	(text ".options method=gear \n.options gmin=1e-9 cshunt=1e-12 \n.options reltol=1e-2 abstol=1e-9 vntol=1e-6 \n.options itl1=300 itl4=300 \n.options maxstep=100p\n.options temp=60\n.tran 100u 1000ms\n.control\nrun\nplot v(Gate) v(Net-_D3-A_) + 0.25 v(Net-_U1A--_)  v(Net-_U1A--_, Net-_D3-A_) v(Comparator)\nplot v(Net-_D9-K_) v(Net-_R7-Pad2_) + 0.25 v(Envelope) v(Output)\nplot v(Envelope) v(Net-_U2C--_) + 0.25 v(Feedback) + 0.35 v(Output) + 0.45\n.endc\n"
+	(text ".options method=gear \n.options gmin=1e-9 cshunt=1e-12 \n.options reltol=1e-2 abstol=1e-9 vntol=1e-6 \n.options itl1=300 itl4=300 \n.options maxstep=100p\n.options temp=60\n.tran 100u 1000ms\n.control\nrun\nplot v(Gate) v(Net-_D3-A_) + 0.25 v(Net-_U1A--_)  v(Net-_U1A--_, Net-_D3-A_) v(Comparator)\nplot v(Net-_D9-K_) v(Net-_Q2-B_) + 0.25 v(Envelope) v(Output)\nplot v(Envelope) v(Net-_U2C--_) + 0.25 v(Feedback) + 0.35 v(Output) + 0.45\nplot v(Net-_D6-A_) v(Net-_D6-K_) v(Net-_R9-Pad2_)\n.endc\n"
 		(exclude_from_sim no)
 		(at 17.272 156.718 0)
@@
 	)
 	(junction
+		(at 147.32 45.72)
+		(diameter 0)
+		(color 0 0 0 0)
+	)
+	(junction
 		(at 215.9 142.24)
 		(diameter 0)
@@
 	(wire
 		(pts
+			(xy 147.32 44.45) (xy 147.32 45.72)
+		)
+		(stroke
+			(width 0)
+			(type default)
+		)
+	)
+	(wire
+		(pts
 			(xy 157.48 132.08) (xy 151.13 132.08)
 		)
@@
 	(wire
 		(pts
+			(xy 147.32 35.56) (xy 147.32 36.83)
+		)
+		(stroke
+			(width 0)
+			(type default)
+		)
+	)
+	(wire
+		(pts
 			(xy 45.72 130.81) (xy 45.72 133.35)
 		)
@@
 		)
 	)
+	(global_label "+v"
+		(shape input)
+		(at 147.32 35.56 90)
+		(fields_autoplaced yes)
+		(effects
+			(font
+				(size 1.27 1.27)
+			)
+			(justify left)
+		)
+		(property "Intersheetrefs" "${INTERSHEET_REFS}"
+			(at 147.32 30.0348 90)
+			(effects
+				(font
+					(size 1.27 1.27)
+				)
+				(justify left)
+				(hide yes)
+			)
+		)
+	)
 	(global_label "Envelope"
 		(shape input)
@@
 					(unit 1)
 				)
+			)
+		)
+	)
+	(symbol
+		(lib_id "Device:R")
+		(at 147.32 40.64 180)
+		(unit 1)
+		(exclude_from_sim no)
+		(in_bom yes)
+		(on_board yes)
+		(dnp no)
+		(property "Reference" "R16"
+			(at 145.288 41.91 90)
+			(effects
+				(font
+					(size 1.27 1.27)
+				)
+				(justify right)
+			)
+		)
+		(property "Value" "10k"
+			(at 149.606 42.418 90)
+			(effects
+				(font
+					(size 1.27 1.27)
+				)
+				(justify right)
+			)
+		)
+		(property "Footprint" ""
+			(at 149.098 40.64 90)
+			(effects
+				(font
+					(size 1.27 1.27)
+				)
+				(hide yes)
+			)
+		)
+		(property "Datasheet" "~"
+			(at 147.32 40.64 0)
+			(effects
+				(font
+					(size 1.27 1.27)
+				)
+				(hide yes)
+			)
+		)
+		(property "Description" "Resistor"
+			(at 147.32 40.64 0)
+			(effects
+				(font
+					(size 1.27 1.27)
+				)
+				(hide yes)
+			)
+		)
+		(pin "2"
+		)
+		(pin "1"
+		)
+		(instances
+			(project "MainBoard"
+				(path "/b7fe592a-70f1-4018-a1e6-02a0fad66ba8"
+					(reference "R16")
+					(unit 1)
+				)

Commit message: checkpoint
Parts:
- removed R16: 10k, symbol Device:R
- C7: value 10uf -> 1uf
- R12: value 47k -> 200k
- RV2: value 100k -> 50k
Connections:
- net Feedback: now also Q1.2 (B), R7.1, U1.5 (+); no longer U1.6 (-)
- new net: R15.2, U1.6 (-)
Other:
- note added: ".options method=gear .options gmin=1e-9 cshunt=1e-12 .options reltol=1e-2 abstol=1e-9 vntol=1e-6 .options itl1=300 itl4=300 .options maxstep=100p .options temp=60 .tran 100u 2500ms .control run *plot v(Gate) v(Net-_D3-A_) + 0.25 v(Net-_U1A--_) v(Net-_U1A--_, Net-_D3-A_) v(Comparator) *plot v(Net-_D9-K_) v(Net-_Q2-B_) + 0.25 v(Envelope) v(Output) *plot v(Envelope) v(Net-_U2C--_) + 0.25 v(Feedback)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"
- note removed: ".options method=gear .options gmin=1e-9 cshunt=1e-12 .options reltol=1e-2 abstol=1e-9 vntol=1e-6 .options itl1=300 itl4=300 .options maxstep=100p .options temp=60 .tran 100u 1000ms .control run plot v(Gate) v(Net-_D3-A_) + 0.25 v(Net-_U1A--_) v(Net-_U1A--_, Net-_D3-A_) v(Comparator) plot v(Net-_D9-K_) v(Net-_Q2-B_) + 0.25 v(Envelope) v(Output) plot v(Envelope) v(Net-_U2C--_) + 0.25 v(Feedback) + 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"
- moved on the sheet: D5, R14, R15, R8, RV2

Commit message: checkpoint
Connections:
- net Feedback: no longer Q1.2 (B)
- net at R15.2, U1.6 (-): now also Q1.2 (B)
Changed lines of the file:
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@@
 		)
 	)
-	(text ".options method=gear \n.options gmin=1e-9 cshunt=1e-12 \n.options reltol=1e-2 abstol=1e-9 vntol=1e-6 \n.options itl1=300 itl4=300 \n.options maxstep=100p\n.options temp=60\n.tran 100u 2500ms\n.control\nrun\n*plot v(Gate) v(Net-_D3-A_) + 0.25 v(Net-_U1A--_)  v(Net-_U1A--_, Net-_D3-A_) v(Comparator)\n*plot v(Net-_D9-K_) v(Net-_Q2-B_) + 0.25 v(Envelope) v(Output)\n*plot v(Envelope) v(Net-_U2C--_) + 0.25 v(Feedback) + 0.35 v(Output) + 0.45\n*plot v(Net-_D6-A_) v(Net-_D6-K_) v(Net-_R9-Pad2_)\nplot v(Net-_Q2-B_) + 0.1 v(Net-_Q2-C_) + 0.2 v(Envelope) + 0.3\n.endc\n"
+	(text ".options method=gear \n.options gmin=1e-9 cshunt=1e-12 \n.options reltol=1e-2 abstol=1e-9 vntol=1e-6 \n.options itl1=300 itl4=300 \n.options maxstep=100p\n.options temp=60\n.tran 100u 2500ms\n.control\nrun\n*plot v(Gate) v(Net-_D3-A_) + 0.25 v(Net-_U1A--_)  v(Net-_U1A--_, Net-_D3-A_) v(Comparator)\n*plot v(Net-_D9-K_) v(Net-_Q2-B_) + 0.25 v(Envelope) v(Output)\n*plot v(Envelope) v(Net-_U2C--_) + 0.25 v(Feedback) + 0.35 v(Output) + 0.45\n*plot v(Net-_D6-A_) v(Net-_D6-K_) v(Net-_R9-Pad2_)\nplot v(Net-_Q2-B_) + 0.1 v(Net-_Q2-C_) + 0.2 v(Envelope) + 0.3 v(Net-_D9-k_)\n.endc\n"
 		(exclude_from_sim no)
 		(at 17.272 156.718 0)
@@
 	)
 	(junction
+		(at 120.65 48.26)
+		(diameter 0)
+		(color 0 0 0 0)
+	)
+	(junction
 		(at 193.04 88.9)
 		(diameter 0)
@@
 	)
 	(junction
-		(at 121.92 66.04)
-		(diameter 0)
-		(color 0 0 0 0)
-	)
-	(junction
 		(at 57.15 50.8)
 		(diameter 0)
@@
 	(wire
 		(pts
+			(xy 120.65 48.26) (xy 120.65 93.98)
+		)
+		(stroke
+			(width 0)
+			(type default)
+		)
+	)
+	(wire
+		(pts
 			(xy 57.15 50.8) (xy 88.9 50.8)
 		)
@@
 	(wire
 		(pts
-			(xy 119.38 48.26) (xy 121.92 48.26)
+			(xy 119.38 48.26) (xy 120.65 48.26)
 		)
 		(stroke
@@
 	(wire
 		(pts
+			(xy 120.65 93.98) (xy 149.86 93.98)
+		)
+		(stroke
+			(width 0)
+			(type default)
+		)
+	)
+	(wire
+		(pts
 			(xy 107.95 123.19) (xy 90.17 123.19)
 		)
@@
 	(wire
 		(pts
-			(xy 121.92 93.98) (xy 121.92 66.04)
-		)
-		(stroke
-			(width 0)
-			(type default)
-		)
-	)
-	(wire
-		(pts
 			(xy 236.22 134.62) (xy 242.57 134.62)
 		)
@@
 	(wire
 		(pts
+			(xy 120.65 48.26) (xy 121.92 48.26)
+		)
+		(stroke
+			(width 0)
+			(type default)
+		)
+	)
+	(wire
+		(pts
 			(xy 134.62 132.08) (xy 134.62 133.35)
 		)
@@
 		)
 		(stroke
-			(width 0)
-			(type default)
-		)
-	)
-	(wire
-		(pts
-			(xy 121.92 93.98) (xy 149.86 93.98)
-		)
-		(stroke

Commit message: checkpoint
Parts:
- RV1, RV3, RV4: value 100k -> 50k
Changed lines of the file:
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@@
 		)
 	)
-	(text ".options method=gear \n.options gmin=1e-9 cshunt=1e-12 \n.options reltol=1e-2 abstol=1e-9 vntol=1e-6 \n.options itl1=300 itl4=300 \n.options maxstep=100p\n.options temp=60\n.tran 100u 2500ms\n.control\nrun\n*plot v(Gate) v(Net-_D3-A_) + 0.25 v(Net-_U1A--_)  v(Net-_U1A--_, Net-_D3-A_) v(Comparator)\n*plot v(Net-_D9-K_) v(Net-_Q2-B_) + 0.25 v(Envelope) v(Output)\n*plot v(Envelope) v(Net-_U2C--_) + 0.25 v(Feedback) + 0.35 v(Output) + 0.45\n*plot v(Net-_D6-A_) v(Net-_D6-K_) v(Net-_R9-Pad2_)\nplot v(Net-_Q2-B_) + 0.1 v(Net-_Q2-C_) + 0.2 v(Envelope) + 0.3 v(Net-_D9-k_)\n.endc\n"
+	(text ".options method=gear \n.options gmin=1e-9 cshunt=1e-12 \n.options reltol=1e-2 abstol=1e-9 vntol=1e-6 \n.options itl1=300 itl4=300 \n.options maxstep=100p\n.options temp=60\n.tran 100u 2500ms\n.control\nrun\n*plot v(Gate) v(Net-_D3-A_) + 0.25 v(Net-_U1A--_)  v(Net-_U1A--_, Net-_D3-A_) v(Comparator)\n*plot v(Net-_D9-K_) v(Net-_Q2-B_) + 0.25 v(Envelope) v(Output)\n*plot v(Envelope) v(Net-_U2C--_) + 0.25 v(Feedback) + 0.35 v(Output) + 0.45\n*plot v(Net-_D6-A_) v(Net-_D6-K_) v(Net-_R9-Pad2_)\nplot  v(Net-_Q1-B_) + 0.2 v(Envelope) + 0.3"
 		(exclude_from_sim no)
 		(at 17.272 156.718 0)
@@
 	)
 	(junction
+		(at 111.76 48.26)
+		(diameter 0)
+		(color 0 0 0 0)
+	)
+	(junction
 		(at 170.18 152.4)
 		(diameter 0)
@@
 	(wire
 		(pts
+			(xy 111.76 38.1) (xy 139.7 38.1)
+		)
+		(stroke
+			(width 0)
+			(type default)
+		)
+	)
+	(wire
+		(pts
 			(xy 121.92 66.04) (xy 124.46 66.04)
 		)
@@
 	(wire
 		(pts
+			(xy 111.76 48.26) (xy 111.76 38.1)
+		)
+		(stroke
+			(width 0)
+			(type default)
+		)
+	)
+	(wire
+		(pts
 			(xy 134.62 135.89) (xy 134.62 138.43)
 		)
@@
 		)
 	)
-	(global_label "Comparator"
-		(shape input)
-		(at 139.7 38.1 90)
-		(fields_autoplaced yes)
-		(effects
-			(font
-				(size 1.27 1.27)
-			)
-			(justify left)
-		)
-		(property "Intersheetrefs" "${INTERSHEET_REFS}"
-			(at 139.7 24.1084 90)
-			(effects
-				(font
-					(size 1.27 1.27)
-				)
-				(justify left)
-				(hide yes)
-			)
-		)
-	)
 	(global_label "Envelope"
 		(shape input)
@@
 			)
 		)
-		(property "Value" "100k"
+		(property "Value" "50k"
 			(at 172.72 63.246 90)
 			(effects
@@
 			)
 		)
-		(property "Sim.Params" "Rtot=100k w=0.5"
+		(property "Sim.Params" "Rtot=100k w=0.2"
 			(at 172.72 66.04 0)
 			(effects
@@
 			)
 		)
-		(property "Value" "100k"
+		(property "Value" "50k"
 			(at 199.39 86.36 90)
 			(effects
@@
 			)
 		)
-		(property "Value" "100k"
+		(property "Value" "50k"
 			(at 199.644 71.882 90)
 			(effects
